File: Blank_Project.kicad_sch (KiCad schematic)
At the start: 11 parts

Commit message: Added a resistor.
Parts:
- added R7: 500R, symbol Device:R
Changed lines of the file:
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@@
+    )
+  )
+  (symbol (lib_id "Device:R") (at 116.84 132.08 0) (unit 1)
+    (in_bom yes) (on_board yes) (dnp no) (fields_autoplaced)
+    (property "Reference" "R7" (at 119.38 131.445 0)
+      (effects (font (size 1.27 1.27)) (justify left))
+    )
+    (property "Value" "500R" (at 119.38 133.985 0)
+      (effects (font (size 1.27 1.27)) (justify left))
+    )
+    (property "Footprint" "" (at 115.062 132.08 90)
+      (effects (font (size 1.27 1.27)) hide)
+    )
+    (property "Datasheet" "~" (at 116.84 132.08 0)
+      (effects (font (size 1.27 1.27)) hide)
+    )
+    (pin "1")
+    (pin "2")
+    (instances
+      (project "Blank_Project"
+        (path "/e41a8201-ef4d-4718-89ef-bc4031c44cb0"
+          (reference "R7") (unit 1)
+        )
+      )
     )
   )

Commit message: Added capacitor.
Parts:
- added C6: 10uF, symbol Device:C_Small
Changed lines of the file:
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@@
 (kicad_sch (version 20230121) (generator eeschema)
   (paper "A4")
+  (symbol (lib_id "Device:C_Small") (at 115.57 143.51 0) (unit 1)
+    (in_bom yes) (on_board yes) (dnp no) (fields_autoplaced)
+    (property "Reference" "C6" (at 118.11 142.8813 0)
+      (effects (font (size 1.27 1.27)) (justify left))
+    )
+    (property "Value" "10uF" (at 118.11 145.4213 0)
+      (effects (font (size 1.27 1.27)) (justify left))
+    )
+    (property "Footprint" "" (at 115.57 143.51 0)
+      (effects (font (size 1.27 1.27)) hide)
+    )
+    (property "Datasheet" "~" (at 115.57 143.51 0)
+      (effects (font (size 1.27 1.27)) hide)
+    )
+    (pin "1")
+    (pin "2")
+    (instances
+      (project "Blank_Project"
+        (path "/e41a8201-ef4d-4718-89ef-bc4031c44cb0"
+          (reference "C6") (unit 1)
+        )
+      )
+    )
+  )
   (symbol (lib_id "Device:R") (at 128.27 132.08 0) (unit 1)
     (in_bom yes) (on_board yes) (dnp no) (fields_autoplaced)

Commit message: Added R8.
Parts:
- added R8: 500R, symbol Device:R
Other:
- moved on the sheet: C6
Changed lines of the file:
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@@
 (kicad_sch (version 20230121) (generator eeschema)
   (paper "A4")
-  (symbol (lib_id "Device:C_Small") (at 115.57 143.51 0) (unit 1)
+  (symbol (lib_id "Device:C_Small") (at 116.84 143.51 0) (unit 1)
     (in_bom yes) (on_board yes) (dnp no) (fields_autoplaced)
-    (property "Reference" "C6" (at 118.11 142.8813 0)
+    (property "Reference" "C6" (at 119.38 142.8813 0)
       (effects (font (size 1.27 1.27)) (justify left))
     )
-    (property "Value" "10uF" (at 118.11 145.4213 0)
+    (property "Value" "10uF" (at 119.38 145.4213 0)
       (effects (font (size 1.27 1.27)) (justify left))
     )
-    (property "Footprint" "" (at 115.57 143.51 0)
+    (property "Footprint" "" (at 116.84 143.51 0)
       (effects (font (size 1.27 1.27)) hide)
     )
-    (property "Datasheet" "~" (at 115.57 143.51 0)
+    (property "Datasheet" "~" (at 116.84 143.51 0)
       (effects (font (size 1.27 1.27)) hide)
     )
@@
         )
       )
+    )
+  )
+  (symbol (lib_id "Device:R") (at 106.68 130.81 0) (unit 1)
+    (in_bom yes) (on_board yes) (dnp no) (fields_autoplaced)
+    (property "Reference" "R8" (at 109.22 130.175 0)
+      (effects (font (size 1.27 1.27)) (justify left))
+    )
+    (property "Value" "500R" (at 109.22 132.715 0)
+      (effects (font (size 1.27 1.27)) (justify left))
+    )
+    (property "Footprint" "" (at 104.902 130.81 90)
+      (effects (font (size 1.27 1.27)) hide)
+    )
+    (property "Datasheet" "~" (at 106.68 130.81 0)
+      (effects (font (size 1.27 1.27)) hide)
+    )
+    (pin "1")
+    (pin "2")
+    (instances
+      (project "Blank_Project"
+        (path "/e41a8201-ef4d-4718-89ef-bc4031c44cb0"
+          (reference "R8") (unit 1)
+        )
+      )
